File: KiCad/ProPrj_SaturnAdapter_2025-11-23.kicad_pcb (KiCad board)
At the start: 2 copper layers, 51.5 x 35.1 mm, 32 parts

Commit message: Rev 0.5 changes | Moving of USB C port next to DB-9/MD connector
Parts:
- moved USB-1 37.1 mm to (128.8, 89.0)
- moved R16 31.0 mm to (137.1, 88.6), turned to 180 degrees
- moved R15 28.9 mm to (137.1, 87.0), turned to 180 degrees
- moved C2 21.0 mm to (136.9, 92.6), turned to 180 degrees
- moved SW1 6.44 mm to (148.2, 86.0)
Routing:
- net EXT5V: track 7.23 -> 17.9 mm, vias 0 -> 2
- net CC2: track 2.95 -> 11.5 mm
- net C+5V: track 34.8 -> 41.1 mm
- net OUT+5V: track 18.5 -> 12.6 mm, vias 4 -> 2
- net CC1: track 2.99 -> 8.27 mm
- net PICO+5V: track 32.3 -> 36.6 mm, vias 2 -> 0
- net LO_D0: track 28.2 -> 29.2 mm, vias 2 -> 0
- net GND: track 2.72 -> 2.89 mm, vias 27 -> 29
Other:
- board size 51.5 x 35.1 mm -> 51.5 x 41.2 mm
- board text added: "REV 0.5"
- board text removed: "REV 0.4"
